File: slider_driver/slider_driver.sch (KiCad schematic (older format))
At the start: 15 parts, among them P1 TOUCH1, P2 TOUCH2, P3 WIPER, P4 IB, P5 IA, P6 +V, P7 GND, U1 L9110, U2 RSA0N11M9A0J

Commit message: added attiny to board
Bit of a feature creep here.  The board is now it's own little self
contained unit that can be accessed using i2c.
Parts:
- removed P1: TOUCH1, symbol CONN_1
- removed P3: WIPER, symbol CONN_1
- removed P4: IB, symbol CONN_1
- removed P5: IA, symbol CONN_1
- added AFF1: 3X7SEGMENTS, symbol 3X7SEGMENTS
- added IC1: ATTINY84A-SS, SO14, symbol ATTINY84A-SS
- added P1, P3: 5_PIN_SOCKET, symbol 5_PIN_SOCKET
- added P4: I2C, ~, symbol I2C
- added P5: ISCP, symbol ISCP
- added P8: +V, symbol CONN_1
- added P9: GND, symbol CONN_1
- added R10, R11, R4, R5, R6, R7, R8, R9: 220, ~, symbol R
- added R12, R13, R14: 500, ~, symbol R
- added SW1: RESET, ~, symbol SW_PUSH
- added U3: BREAK_CONNECTION, symbol BREAK_CONNECTION
- added U4, U5: 74HC595-16-PIN, ~, symbol 74HC595-16-PIN
- P2: value TOUCH2 -> NEOPIXEL
Connections:
- net labels added: +12V
- wire segments 34 -> 198
