File: Circuit/slider_driver.sch (KiCad schematic (older format))
At the start: 34 parts, among them IC1 ATTINY84A-SS, P1 5_PIN_SOCKET, P2 NEOPIXEL, P3 5_PIN_SOCKET, P4 I2C, P5 ISCP, P6 +V, P7 GND, P8 +V, P9 GND, SW1 RESET, U1 L9110, U2 RSA0N11M9A0J, U3 BREAK_CONNECTION, U4 74HC595-16-PIN, U5 74HC595-16-PIN

Commit message: fixed pin for iscp port
Total screw up there.
Parts:
- added D1: LED, ~, symbol LED
- added R15: 1K, ~, symbol R
Connections:
- wire segments 198 -> 201
Changed lines of the file:
@@
 Sheet 1 1
 Title ""
-Date "25 jan 2014"
+Date "1 mar 2014"
 Rev ""
 Comp ""
@@
 $EndComp
 $Comp
-L +5V #PWR01
+L +5V #PWR3
 U 1 1 52D16BE2
 P 2000 1300
-F 0 "#PWR01" H 2000 1390 20  0001 C CNN
+F 0 "#PWR3" H 2000 1390 20  0001 C CNN
 F 1 "+5V" H 2000 1390 30  0000 C CNN
 F 2 "" H 2000 1300 60  0000 C CNN
@@
 $EndComp
 $Comp
-L GND #PWR02
+L GND #PWR4
 U 1 1 52D16BF1
 P 2000 2050
-F 0 "#PWR02" H 2000 2050 30  0001 C CNN
+F 0 "#PWR4" H 2000 2050 30  0001 C CNN
 F 1 "GND" H 2000 1980 30  0001 C CNN
 F 2 "" H 2000 2050 60  0000 C CNN
@@
 $EndComp
 $Comp
-L +5V #PWR03
+L +5V #PWR9
 U 1 1 52D173E0
 P 6400 2150
-F 0 "#PWR03" H 6400 2240 20  0001 C CNN
+F 0 "#PWR9" H 6400 2240 20  0001 C CNN
 F 1 "+5V" H 6400 2240 30  0000 C CNN
 F 2 "" H 6400 2150 60  0000 C CNN
@@
 Connection ~ 5700 3100
 $Comp
-L GND #PWR04
+L GND #PWR8
 U 1 1 52D17AC5
 P 5700 2250
-F 0 "#PWR04" H 5700 2250 30  0001 C CNN
+F 0 "#PWR8" H 5700 2250 30  0001 C CNN
 F 1 "GND" H 5700 2180 30  0001 C CNN
 F 2 "" H 5700 2250 60  0000 C CNN
@@
 $EndComp
 $Comp
-L +5V #PWR05
+L +5V #PWR5
 U 1 1 52D17B46
 P 3050 4700
-F 0 "#PWR05" H 3050 4790 20  0001 C CNN
+F 0 "#PWR5" H 3050 4790 20  0001 C CNN
 F 1 "+5V" H 3050 4790 30  0000 C CNN
 F 2 "" H 3050 4700 60  0000 C CNN
@@
 	3050 4200 3050 4700
 $Comp
-L GND #PWR06
+L GND #PWR6
 U 1 1 52D17BC6
 P 3400 4750
-F 0 "#PWR06" H 3400 4750 30  0001 C CNN
+F 0 "#PWR6" H 3400 4750 30  0001 C CNN
 F 1 "GND" H 3400 4680 30  0001 C CNN
 F 2 "" H 3400 4750 60  0000 C CNN
@@
 Connection ~ 3050 4600
 $Comp
-L +12V #PWR07
+L +12V #PWR7
 U 1 1 52E2490E
 P 3750 2250
-F 0 "#PWR07" H 3750 2200 20  0001 C CNN
+F 0 "#PWR7" H 3750 2200 20  0001 C CNN
 F 1 "+12V" H 3750 2350 30  0000 C CNN
 F 2 "" H 3750 2250 60  0000 C CNN
@@
 $EndComp
 $Comp
-L GND #PWR08
+L GND #PWR10
 U 1 1 52E38A27
 P 9650 2250
-F 0 "#PWR08" H 9650 2250 30  0001 C CNN
+F 0 "#PWR10" H 9650 2250 30  0001 C CNN
 F 1 "GND" H 9650 2180 30  0001 C CNN
 F 2 "" H 9650 2250 60  0000 C CNN
@@
 	9650 2650 9650 2250
 $Comp
-L +5V #PWR09
+L +5V #PWR11
 U 1 1 52E38A90
 P 9650 3300
-F 0 "#PWR09" H 9650 3390 20  0001 C CNN
+F 0 "#PWR11" H 9650 3390 20  0001 C CNN
 F 1 "+5V" H 9650 3390 30  0000 C CNN
 F 2 "" H 9650 3300 60  0000 C CNN
@@
 $EndComp
 Wire Wire Line
-	9450 2650 9450 2250
+	9450 2250 9450 2950
 Wire Wire Line
 	9450 2250 8750 2250
@@
 	9450 3850 9450 4200
 Wire Wire Line
-	9150 4200 10000 4200
-Wire Wire Line
-	10000 4200 10000 5600
+	10000 2950 10000 5600
 Wire Wire Line
 	10000 5600 9250 5600
@@
 Wire Wire Line
 	3600 2400 3600 2800
+$Comp
+L +5V #PWR1
+U 1 1 530DF118
+P 1500 1300
+F 0 "#PWR1" H 1500 1390 20  0001 C CNN
+F 1 "+5V" H 1500 1390 30  0000 C CNN
+F 2 "" H 1500 1300 60  0000 C CNN
+F 3 "" H 1500 1300 60  0000 C CNN
+	1    1500 1300
+	1    0    0    -1
+$EndComp
+$Comp
+L R R15
+U 1 1 530DF127
+P 1500 1650
+F 0 "R15" V 1580 1650 40  0000 C CNN
+F 1 "1K" V 1507 1651 40  0000 C CNN
+F 2 "~" V 1430 1650 30  0000 C CNN
+F 3 "~" H 1500 1650 30  0000 C CNN
+	1    1500 1650
+	1    0    0    -1
+$EndComp
+$Comp
+L LED D1
+U 1 1 530DF147
+P 1500 2100
+F 0 "D1" H 1500 2200 50  0000 C CNN
+F 1 "LED" H 1500 2000 50  0000 C CNN
+F 2 "~" H 1500 2100 60  0000 C CNN
+F 3 "~" H 1500 2100 60  0000 C CNN
+	1    1500 2100
+	0    1    1    0
+$EndComp
+$Comp
+L GND #PWR2
+U 1 1 530DF16F
+P 1500 2450
+F 0 "#PWR2" H 1500 2450 30  0001 C CNN
+F 1 "GND" H 1500 2380 30  0001 C CNN
+F 2 "" H 1500 2450 60  0000 C CNN
+F 3 "" H 1500 2450 60  0000 C CNN
+	1    1500 2450
+	1    0    0    -1
+$EndComp
+Wire Wire Line
+	1500 2450 1500 2300
+Wire Wire Line
+	1500 1400 1500 1300
+Wire Wire Line
+	9150 4200 9450 4200
+Wire Wire Line
+	9450 2950 10000 2950
 $EndSCHEMATC

Commit message: Extra pins Re Bug #3
Parts:
- added P10: +V, symbol CONN_1
- added P11: GND, symbol CONN_1
Changed lines of the file:
@@
 Sheet 1 1
 Title ""
-Date "1 mar 2014"
+Date "12 mar 2014"
 Rev ""
 Comp ""
@@
 Wire Wire Line
 	9450 2950 10000 2950
+$Comp
+L CONN_1 P11
+U 1 1 53203875
+P 5550 2650
+F 0 "P11" H 5630 2650 40  0000 L CNN
+F 1 "GND" H 5550 2705 30  0001 C CNN
+F 2 "" H 5550 2650 60  0000 C CNN
+F 3 "" H 5550 2650 60  0000 C CNN
+	1    5550 2650
+	-1   0    0    1
+$EndComp
+$Comp
+L CONN_1 P10
+U 1 1 5320387B
+P 3900 2500
+F 0 "P10" H 3980 2500 40  0000 L CNN
+F 1 "+V" H 3900 2555 30  0001 C CNN
+F 2 "" H 3900 2500 60  0000 C CNN
+F 3 "" H 3900 2500 60  0000 C CNN
+	1    3900 2500
+	1    0    0    -1
+$EndComp
+Connection ~ 5700 2650
+Connection ~ 3750 2500
 $EndSCHEMATC

Commit message: Updated board to support max chip
Parts:
- removed AFF1: 3X7SEGMENTS, symbol 3X7SEGMENTS
- removed P10, P6, P8: +V, symbol CONN_1
- removed P11, P7, P9: GND, symbol CONN_1
- removed P2: NEOPIXEL, symbol CONN_1
- removed P3: 5_PIN_SOCKET, symbol 5_PIN_SOCKET
- removed P4: I2C, ~, symbol I2C
- removed P5: ISCP, symbol ISCP
- removed R10, R11, R6, R7, R8, R9: 220, ~, symbol R
- removed R12, R13, R14: 500, ~, symbol R
- removed SW1: RESET, ~, symbol SW_PUSH
- removed U1: L9110, ~, symbol L9110
- removed U3: BREAK_CONNECTION, symbol BREAK_CONNECTION
- removed U4, U5: 74HC595-16-PIN, ~, symbol 74HC595-16-PIN
- added AFF1: 3X7SEGMENTS_1, ~, symbol 3X7SEGMENTS_1
- added C4: 0.1uf, ~, symbol C
- added C5: 10uf, ~, symbol C
- added K1: Neopixel, symbol CONN_3
- added K2: PWR, symbol CONN_3
- added P2: 5_PIN_SOCKET, symbol 5_PIN_SOCKET
- added P3: ISCP, symbol ISCP
- added P4: Bridge, symbol CONN_2
- added U1: MAX7219, symbol MAX7219
- added U3: L9110, ~, symbol L9110
- R1: value 10k -> 28
- R4, R5: value 220 -> 10k
Connections:
- net labels added: IA, IB, MISO, MOSI, Motor_1, Motor_2, RCLK, RESET, Receive, SCK, SER, SRCLK, Send, Touch, Wiper
- wire segments 201 -> 51
- no-connect marks 0 -> 8
Other:
- moved on the sheet: C1, C2, D1, IC1, R15, R3

Commit message: Some changes that I guess were important at some point
Parts:
- AFF1: symbol 3X7SEGMENTS_1 -> 3x7SEGMENTS_1
- C1, C2, C3, C4, C5: symbol C -> C-RESCUE-slider_driver
- D1: symbol LED -> LED-RESCUE-slider_driver
- P1, P2: symbol 5_PIN_SOCKET -> 5_pin_socket
- R1, R15, R2, R3, R4, R5: symbol R -> R-RESCUE-slider_driver
Changed lines of the file:
@@
 EESchema Schematic File Version 2
+LIBS:slider_driver-rescue
 LIBS:slider_driver
 LIBS:power
@@
 LIBS:memory
 LIBS:xilinx
-LIBS:special
 LIBS:microcontrollers
 LIBS:dsp
@@
 LIBS:w_logic
 LIBS:mages_mega
-LIBS:slider_driver-cache
-EELAYER 27 0
+EELAYER 25 0
 EELAYER END
 $Descr A4 11693 8268
@@
 $EndDescr
 $Comp
-L C C1
+L C-RESCUE-slider_driver C1
 U 1 1 52D16BBC
 P 900 800
@@
 $EndComp
 $Comp
-L GND #PWR4
+L GND-RESCUE-slider_driver #PWR4
 U 1 1 52D16BF1
 P 900 1000
@@
 $EndComp
 $Comp
-L C C2
+L C-RESCUE-slider_driver C2
 U 1 1 52D16BFE
 P 1100 800
@@
 	1100 600  900  600
 $Comp
-L R R3
+L R-RESCUE-slider_driver R3
 U 1 1 52D2122A
 P 7100 1200
@@
 $EndComp
 $Comp
-L GND #PWR32
+L GND-RESCUE-slider_driver #PWR32
 U 1 1 52E38A27
 P 11000 900
@@
 $EndComp
 $Comp
-L R R15
+L R-RESCUE-slider_driver R15
 U 1 1 530DF127
 P 650 850
@@
 $EndComp
 $Comp
-L LED D1
+L LED-RESCUE-slider_driver D1
 U 1 1 530DF147
 P 650 1300
@@
 $EndComp
 $Comp
-L GND #PWR2
+L GND-RESCUE-slider_driver #PWR2
 U 1 1 530DF16F
 P 650 1500
@@
 $EndComp
 $Comp
-L GND #PWR31
+L GND-RESCUE-slider_driver #PWR31
 U 1 1 558EB6FB
 P 10400 3000
@@
 $EndComp
 $Comp
-L GND #PWR27
+L GND-RESCUE-slider_driver #PWR27
 U 1 1 558EB919
 P 9900 4500
@@
 $EndComp
 $Comp
-L GND #PWR26
+L GND-RESCUE-slider_driver #PWR26
 U 1 1 558EB91F
 P 9900 3500
@@
 $EndComp
 $Comp
-L R R4
+L R-RESCUE-slider_driver R4
 U 1 1 558EB931
 P 10100 3550
@@
 $EndComp
 $Comp
-L R R5
+L R-RESCUE-slider_driver R5
 U 1 1 558EB937
 P 10100 4450
@@
 $EndComp
 $Comp
-L GND #PWR19
+L GND-RESCUE-slider_driver #PWR19
 U 1 1 558EBB0B
 P 6650 2500
@@
 	6650 2250 6650 2200
 $Comp
-L C C3
+L C-RESCUE-slider_driver C3
 U 1 1 558EBC5A
 P 8050 4000
@@
 Connection ~ 7350 1200
 $Comp
-L R R2
+L R-RESCUE-slider_driver R2
 U 1 1 558EBDEA
 P 8550 900
@@
 Send
 $Comp
-L 5_PIN_SOCKET P2
+L 5_pin_socket P2
 U 1 1 558EBF59
 P 4650 900
@@
 $EndComp
 $Comp
-L GND #PWR18
+L GND-RESCUE-slider_driver #PWR18
 U 1 1 558EC04D
 P 4550 1300
@@
 $EndComp
 $Comp
-L GND #PWR14
+L GND-RESCUE-slider_driver #PWR14
 U 1 1 558EC4EE
 P 3050 5500
@@
 $EndComp
 $Comp
-L 3X7SEGMENTS_1 AFF1
+L 3x7SEGMENTS_1 AFF1
 U 1 1 558EC889
 P 4600 4950
@@
 NoConn ~ 2700 4400
 $Comp
-L R R1
+L R-RESCUE-slider_driver R1
 U 1 1 558EC92B
 P 2700 3450
@@
 $EndComp
 $Comp
-L 5_PIN_SOCKET P1
+L 5_pin_socket P1
 U 1 1 558EC94A
 P 2200 3800
@@
 $EndComp
 $Comp
-L GND #PWR8
+L GND-RESCUE-slider_driver #PWR8
 U 1 1 558EC950
 P 2100 4200
@@
 $EndComp
 $Comp
-L GND #PWR22
+L GND-RESCUE-slider_driver #PWR22
 U 1 1 558ECE46
 P 7900 1000
@@
 $EndComp
 $Comp
-L GND #PWR10
+L GND-RESCUE-slider_driver #PWR10
 U 1 1 559116BD
 P 2550 1150
@@
 $EndComp
 $Comp
-L C C4
+L C-RESCUE-slider_driver C4
 U 1 1 55911883
 P 1950 5150
@@
 $EndComp
 $Comp
-L GND #PWR6
+L GND-RESCUE-slider_driver #PWR6
 U 1 1 5591188F
 P 1950 5350
@@
 $EndComp
 $Comp
-L C C5
+L C-RESCUE-slider_driver C5
 U 1 1 55911895
 P 2150 5150
